File: tugas-akhir.kicad_sch (KiCad schematic)
At the start: 30 parts, among them J1 Conn_01x02_Socket, J2 Conn_01x02_Pin (solenoid lini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, K1 Relay_SPDT, M1 Stepper_Motor_bipolar / Nema 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, M2 Stepper_Motor_bipolar / Nema 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, M3 Stepper_Motor_bipolar / Nema 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, Q1 2N3904, U1 ESP32-DEVKIT-V1, U2 DCDC_StepDown_LM2596, U3 TMC2208_SILENTSTEPSTICK, U4 TMC2208_SILENTSTEPSTICK, U5 TMC2208_SILENTSTEPSTICK

Commit message: route stepper driver
Connections:
- net at U1.3 (D15): no longer R3.1
Changed lines of the file:
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@@
-	(wire
-		(pts
-			(xy 81.28 118.11) (xy 81.28 123.19)
-		)
-		(stroke
-			(width 0)
-			(type default)
-		)
-	)
 	(wire
 		(pts
@@
 	(wire
 		(pts
-			(xy 105.41 104.14) (xy 105.41 118.11)
-		)
-		(stroke
-			(width 0)
-			(type default)
-		)
-	)
-	(wire
-		(pts
 			(xy 161.29 118.11) (xy 245.11 118.11)
 		)
@@
 	(wire
 		(pts
-			(xy 81.28 123.19) (xy 69.85 123.19)
-		)
-		(stroke
-			(width 0)
-			(type default)
-		)
-	)
-	(wire
-		(pts
 			(xy 224.79 93.98) (xy 205.74 93.98)
 		)
@@
 	(wire
 		(pts
-			(xy 105.41 118.11) (xy 81.28 118.11)
-		)
-		(stroke
-			(width 0)
-			(type default)
-		)
-	)
-	(wire
-		(pts
 			(xy 170.18 81.28) (xy 163.83 81.28)
 		)
@@
 		)
 		(stroke
-			(width 0)
-			(type default)
-		)
-	)
-	(wire
-		(pts
-			(xy 120.65 104.14) (xy 105.41 104.14)
-		)
-		(stroke

Commit message: feat: new route
Connections:
- net at U3.JP1_8 (EN): now also U1.11 (D21); no longer U1.27 (D12)
- net at R6.1: no longer U1.9 (D18)
- net at U4.JP1_1 (DIR): now also U1.9 (D18); no longer U1.11 (D21)
- net at U1.28 (D13): no longer U4.JP1_8 (EN)
- net at U1.3 (D15): now also R3.1
- net at U1.8 (D5): now also U4.JP1_8 (EN)

Commit message: finish pcb route
Parts:
- D3: footprint Diode_THT:D_DO-201AD_P15.24mm_Horizontal -> Diode_THT:D_DO-41_SOD81_P7.62mm_Horizontal
Connections:
- net at U3.JP1_6 (MS2), U4.JP1_6 (MS2), U5.JP1_6 (MS2): now also U1.24 (D26); no longer U1.22 (D33)
- net at U3.JP1_7 (MS1), U4.JP1_7 (MS1), U5.JP1_7 (MS1): now also U1.23 (D25); no longer U1.21 (D32)
- net at R5.1: now also U1.28 (D13); no longer U1.19 (D34)
- net at R6.1: now also U1.27 (D12)
- net at S1.1: now also U1.8 (D5); no longer U1.25 (D27)
- net at U1.10 (D19): now also U4.JP1_8 (EN); no longer U4.JP1_2 (STEP)
- net at U1.20 (D35): now also U4.JP1_2 (STEP); no longer R4.1
- net at S3.1: now also U1.9 (D18); no longer U1.23 (D25)
- net at S2.1: now also U1.7 (TX2); no longer U1.24 (D26)
- net at U5.JP1_8 (EN): now also U1.25 (D27); no longer U1.26 (D14)
- net at R3.1: now also U1.26 (D14); no longer U1.3 (D15)
- net at U5.JP1_2 (STEP): now also U1.22 (D33); no longer U1.4 (D2)
- net at U5.JP1_1 (DIR): now also U1.21 (D32); no longer U1.5 (D4)
- net at U4.JP1_1 (DIR): now also U1.19 (D34); no longer U1.9 (D18)
- new net: R4.1, U1.3 (D15)

Commit message: new pcb route
Parts:
- Q1: footprint Package_TO_SOT_THT:TO-92_Inline -> Package_TO_SOT_THT:TO-92_Inline_Wide
Connections:
- net at S1.1: now also U1.4 (D2); no longer U1.8 (D5)
- net at U1.19 (D34): no longer U4.JP1_1 (DIR)
- net at U1.20 (D35): no longer U4.JP1_2 (STEP)
- net at U1.26 (D14): now also R4.1; no longer R3.1
- net at U1.3 (D15): no longer R4.1
- net at U1.5 (D4): now also S2.1
- net at U1.6 (RX2): now also U4.JP1_1 (DIR)
- net at U1.7 (TX2): now also U4.JP1_2 (STEP); no longer S2.1
- new net: R3.1, U1.8 (D5)

Commit message: change size of resistor and terminal block
Parts:
- J1: footprint TerminalBlock_Phoenix:TerminalBlock_Phoenix_MKDS-1,5-2-5.08_1x02_P5.08mm_Horizontal -> TerminalBlock_Phoenix:TerminalBlock_Phoenix_PT-1,5-2-3.5-H_1x02_P3.50mm_Horizontal
- R1, R2, R3, R4, R5, R6: footprint Resistor_THT:R_Axial_DIN0204_L3.6mm_D1.6mm_P5.08mm_Horizontal -> Resistor_THT:R_Axial_DIN0204_L3.6mm_D1.6mm_P7.62mm_Horizontal
Changed lines of the file:
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@@
 			)
 		)
-		(property "Footprint" "Resistor_THT:R_Axial_DIN0204_L3.6mm_D1.6mm_P5.08mm_Horizontal"
+		(property "Footprint" "Resistor_THT:R_Axial_DIN0204_L3.6mm_D1.6mm_P7.62mm_Horizontal"
 			(at 249.682 73.66 90)
 			(effects
@@
 			)
 		)
-		(property "Footprint" "Resistor_THT:R_Axial_DIN0204_L3.6mm_D1.6mm_P5.08mm_Horizontal"
+		(property "Footprint" "Resistor_THT:R_Axial_DIN0204_L3.6mm_D1.6mm_P7.62mm_Horizontal"
 			(at 87.122 101.6 90)
 			(effects
@@
 			)
 		)
-		(property "Footprint" "Resistor_THT:R_Axial_DIN0204_L3.6mm_D1.6mm_P5.08mm_Horizontal"
+		(property "Footprint" "Resistor_THT:R_Axial_DIN0204_L3.6mm_D1.6mm_P7.62mm_Horizontal"
 			(at 250.952 29.21 90)
 			(effects
@@
 			)
 		)
-		(property "Footprint" "Resistor_THT:R_Axial_DIN0204_L3.6mm_D1.6mm_P5.08mm_Horizontal"
+		(property "Footprint" "Resistor_THT:R_Axial_DIN0204_L3.6mm_D1.6mm_P7.62mm_Horizontal"
 			(at 65.532 101.6 90)
 			(effects
@@
 			)
 		)
-		(property "Footprint" "Resistor_THT:R_Axial_DIN0204_L3.6mm_D1.6mm_P5.08mm_Horizontal"
+		(property "Footprint" "Resistor_THT:R_Axial_DIN0204_L3.6mm_D1.6mm_P7.62mm_Horizontal"
 			(at 66.04 121.412 90)
 			(effects
@@
 			)
 		)
-		(property "Footprint" "Resistor_THT:R_Axial_DIN0204_L3.6mm_D1.6mm_P5.08mm_Horizontal"
+		(property "Footprint" "Resistor_THT:R_Axial_DIN0204_L3.6mm_D1.6mm_P7.62mm_Horizontal"
 			(at 248.412 119.38 90)
 			(effects
@@
 			)
 		)
-		(property "Footprint" "TerminalBlock_Phoenix:TerminalBlock_Phoenix_MKDS-1,5-2-5.08_1x02_P5.08mm_Horizontal"
+		(property "Footprint" "TerminalBlock_Phoenix:TerminalBlock_Phoenix_PT-1,5-2-3.5-H_1x02_P3.50mm_Horizontal"
 			(at 95.25 86.36 0)
 			(effects

Commit message: minor revision
Parts:
- C1, C2, C3: footprint Capacitor_THT:C_Radial_D8.0mm_H11.5mm_P3.50mm -> Capacitor_THT:CP_Radial_D8.0mm_P3.50mm
- D3: value D -> 1N4007
Changed lines of the file:
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@@
 			)
 		)
-		(property "Footprint" "Capacitor_THT:C_Radial_D8.0mm_H11.5mm_P3.50mm"
+		(property "Footprint" "Capacitor_THT:CP_Radial_D8.0mm_P3.50mm"
 			(at 214.63 77.47 0)
 			(effects
@@
 			)
 		)
-		(property "Footprint" "Capacitor_THT:C_Radial_D8.0mm_H11.5mm_P3.50mm"
+		(property "Footprint" "Capacitor_THT:CP_Radial_D8.0mm_P3.50mm"
 			(at 215.9 25.4 0)
 			(effects
@@
 			)
 		)
-		(property "Value" "D"
+		(property "Value" "1N4007"
 			(at 62.23 106.6799 90)
 			(effects
@@
 			)
 		)
-		(property "Footprint" "Capacitor_THT:C_Radial_D8.0mm_H11.5mm_P3.50mm"
+		(property "Footprint" "Capacitor_THT:CP_Radial_D8.0mm_P3.50mm"
 			(at 214.63 125.73 0)
 			(effects

Commit message: update driver routes
Connections:
- net at U3.JP1_3 (CLK): now also U3.JP1_4 (PDN/UART1)
- net at U3.JP1_5 (NC): now also D3.1 (K), K1.2, R1.1, R2.1, S1.3, S2.3, S3.3, U1.1 (3V3), U3.JP2_7 (VIO), U4.JP1_5 (NC), U4.JP2_7 (VIO), U5.JP1_5 (NC), U5.JP2_7 (VIO)
- net at U5.JP1_3 (CLK): now also U5.JP1_4 (PDN/UART1)
- net at U4.JP1_3 (CLK): now also U4.JP1_4 (PDN/UART1)
Changed lines of the file:
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@@
 	(title_block
 		(title "IoT Liquid Dispensing Iodium-131 Capsules")
-		(date "2024-05-01")
-		(rev "4")
+		(date "2024-05-20")
+		(rev "5")
 	)
 	(junction
@@
 	)
 	(junction
+		(at 168.91 146.05)
+		(diameter 0)
+		(color 0 0 0 0)
+	)
+	(junction
 		(at 212.09 19.05)
 		(diameter 0)
@@
 	)
 	(junction
+		(at 166.37 66.04)
+		(diameter 0)
+		(color 0 0 0 0)
+	)
+	(junction
 		(at 154.94 93.98)
 		(diameter 0)
@@
 	)
 	(junction
+		(at 168.91 99.06)
+		(diameter 0)
+		(color 0 0 0 0)
+	)
+	(junction
 		(at 212.09 121.92)
 		(diameter 0)
@@
 	(wire
 		(pts
+			(xy 170.18 104.14) (xy 170.18 106.68)
+		)
+		(stroke
+			(width 0)
+			(type default)
+		)
+	)
+	(wire
+		(pts
 			(xy 67.31 97.79) (xy 88.9 97.79)
 		)
@@
 	(wire
 		(pts
+			(xy 166.37 66.04) (xy 168.91 66.04)
+		)
+		(stroke
+			(width 0)
+			(type default)
+		)
+	)
+	(wire
+		(pts
 			(xy 226.06 52.07) (xy 226.06 48.26)
 		)
@@
 	(wire
 		(pts
+			(xy 168.91 99.06) (xy 170.18 99.06)
+		)
+		(stroke
+			(width 0)
+			(type default)
+		)
+	)
+	(wire
+		(pts
 			(xy 156.21 128.27) (xy 170.18 128.27)
 		)
@@
 	(wire
 		(pts
+			(xy 170.18 151.13) (xy 170.18 153.67)
+		)
+		(stroke
+			(width 0)
+			(type default)
+		)
+	)
+	(wire
+		(pts
 			(xy 161.29 118.11) (xy 245.11 118.11)
 		)
@@
 	(wire
 		(pts
+			(xy 170.18 55.88) (xy 170.18 58.42)
+		)
+		(stroke
+			(width 0)
+			(type default)
+		)
+	)
+	(wire
+		(pts
 			(xy 38.1 96.52) (xy 34.29 96.52)
 		)
@@
 	(wire
 		(pts
-			(xy 168.91 113.03) (xy 168.91 162.56)
+			(xy 168.91 113.03) (xy 168.91 146.05)
 		)
 		(stroke
@@
 	(wire
 		(pts
-			(xy 168.91 66.04) (xy 168.91 113.03)
+			(xy 168.91 66.04) (xy 168.91 99.06)
 		)
 		(stroke
@@
 	(wire
 		(pts
+			(xy 168.91 99.06) (xy 168.91 113.03)
+		)
+		(stroke
+			(width 0)
+			(type default)
+		)
+	)
+	(wire
+		(pts
 			(xy 219.71 81.28) (xy 219.71 33.02)
 		)
@@
 	(wire
 		(pts
+			(xy 166.37 50.8) (xy 166.37 66.04)
+		)
+		(stroke
+			(width 0)
+			(type default)
+		)
+	)
+	(wire
+		(pts
 			(xy 245.11 134.62) (xy 245.11 118.11)
 		)
@@
 	(wire
 		(pts
+			(xy 168.91 146.05) (xy 168.91 162.56)
+		)
+		(stroke
+			(width 0)
+			(type default)
+		)
+	)
+	(wire
+		(pts
 			(xy 147.32 33.02) (xy 147.32 55.88)
 		)
@@
 	(wire
 		(pts
+			(xy 170.18 50.8) (xy 166.37 50.8)
+		)
+		(stroke
+			(width 0)
+			(type default)
+		)
+	)
+	(wire
+		(pts
 			(xy 250.19 134.62) (xy 245.11 134.62)
 		)
@@
 	(wire
 		(pts
-			(xy 157.48 66.04) (xy 168.91 66.04)
+			(xy 157.48 66.04) (xy 166.37 66.04)
 		)
 		(stroke
@@
 		)
 		(stroke
+			(width 0)
+			(type default)
+		)
+	)
+	(wire
+		(pts
+			(xy 168.91 146.05) (xy 170.18 146.05)
+		)
+		(stroke
